Commit message: added teleop

File: install/thor_urdf/share/thor_urdf/urdf/thor.urdf.xacro (robot description, xacro)
@@ -1,15 +1,10 @@
 <?xml version="1.0"?>
 <robot xmlns:xacro="http://www.ros.org/wiki/xacro" name="thor_arm">
-    <!-- Load Simulated or Real Hardware Interfaces -->
     <xacro:arg name="is_sim" default="true"/>
-    <!-- Include Gazebo Parameters -->
     <xacro:include filename="$(find thor_urdf)/urdf/thor_gazebo.xacro" />
-    <!-- Include ros2_control Plugins -->
     <xacro:include filename="$(find thor_urdf)/urdf/thor_arm.ros2_control.xacro" />
-    <!-- Useful XACRO Variables (Properties) -->
     <xacro:property name="PI" value="3.14159265359" />
     <xacro:property name="effort" value="4.0" />
     <xacro:property name="velocity" value="1.0" />
-    <!-- Useful Macros -->
     <xacro:macro name="default_inertial" params="mass">
         <inertial>
@@ -21,5 +16,5 @@
         </inertial>
     </xacro:macro>
-    <!-- Links -->
+    <!-- LINKS -->
     <link name="world"/>
     <link name="base_link">
@@ -147,7 +142,7 @@
         <visual>
             <origin xyz="0 0 0" rpy="0 0 -${PI / 2}"/>
-        <geometry>
-            <mesh filename="package://thor_urdf/meshes/Art6.dae" scale="0.001 0.001 0.001" />
-        </geometry>
+            <geometry>
+                <mesh filename="package://thor_urdf/meshes/Art6.dae" scale="0.001 0.001 0.001" />
+            </geometry>
         </visual>
         <collision>
@@ -158,5 +153,4 @@
         </collision>
     </link>
-    <!-- Electromagnet End Effector -->
     <link name="electromagnet_mount">
         <xacro:default_inertial mass="0.2"/>
@@ -195,5 +189,160 @@
         </collision>
     </link>
-    <!-- Overhead Camera System (floating above workspace) -->
+    <link name="table_base">
+        <inertial>
+            <origin xyz="0 0 0" rpy="0 0 0"/>
+            <mass value="10.0" />
+            <inertia ixx="0.147" ixy="0.0" ixz="0.0"
+                     iyy="0.213" iyz="0.0"
+                     izz="0.347" />
+        </inertial>
+        <visual>
+            <origin xyz="0 0 0" rpy="0 0 0"/>
+            <geometry>
+                <box size="0.5 0.4 0.04"/>
+            </geometry>
+            <material name="table_material">
+                <color rgba="0.6 0.4 0.2 1.0"/>
+            </material>
+        </visual>
+        <collision>
+            <origin xyz="0 0 0" rpy="0 0 0"/>
+            <geometry>
+                <box size="0.5 0.4 0.04"/>
+            </geometry>
+        </collision>
+    </link>
+    <link name="table_leg_1">
+        <inertial>
+            <origin xyz="0 0 0" rpy="0 0 0"/>
+            <mass value="2.0" />
+            <inertia ixx="0.0085" ixy="0.0" ixz="0.0"
+                     iyy="0.0085" iyz="0.0"
+                     izz="0.0006" />
+        </inertial>
+        <visual>
+            <origin xyz="0 0 0" rpy="0 0 0"/>
+            <geometry>
+                <cylinder radius="0.015" length="0.25"/>
+            </geometry>
+            <material name="leg_material">
+                <color rgba="0.4 0.3 0.1 1.0"/>
+            </material>
+        </visual>
+        <collision>
+            <origin xyz="0 0 0" rpy="0 0 0"/>
+            <geometry>
+                <cylinder radius="0.015" length="0.25"/>
+            </geometry>
+        </collision>
+    </link>
+    <link name="table_leg_2">
+        <inertial>
+            <origin xyz="0 0 0" rpy="0 0 0"/>
+            <mass value="2.0" />
+            <inertia ixx="0.0085" ixy="0.0" ixz="0.0"
+                     iyy="0.0085" iyz="0.0"
+                     izz="0.0006" />
+        </inertial>
+        <visual>
+            <origin xyz="0 0 0" rpy="0 0 0"/>
+            <geometry>
+                <cylinder radius="0.015" length="0.25"/>
+            </geometry>
+            <material name="leg_material">
+                <color rgba="0.4 0.3 0.1 1.0"/>
+            </material>
+        </visual>
+        <collision>
+            <origin xyz="0 0 0" rpy="0 0 0"/>
+            <geometry>
+                <cylinder radius="0.015" length="0.25"/>
+            </geometry>
+        </collision>
+    </link>
+    <link name="table_leg_3">
+        <inertial>
+            <origin xyz="0 0 0" rpy="0 0 0"/>
+            <mass value="2.0" />
+            <inertia ixx="0.0085" ixy="0.0" ixz="0.0"
+                     iyy="0.0085" iyz="0.0"
+                     izz="0.0006" />
+        </inertial>
+        <visual>
+            <origin xyz="0 0 0" rpy="0 0 0"/>
+            <geometry>
+                <cylinder radius="0.015" length="0.25"/>
+            </geometry>
+            <material name="leg_material">
+                <color rgba="0.4 0.3 0.1 1.0"/>
+            </material>
+        </visual>
+        <collision>
+            <origin xyz="0 0 0" rpy="0 0 0"/>
+            <geometry>
+                <cylinder radius="0.015" length="0.25"/>
+            </geometry>
+        </collision>
+    </link>
+    <link name="table_leg_4">
+        <inertial>
+            <origin xyz="0 0 0" rpy="0 0 0"/>
+            <mass value="2.0" />
+            <inertia ixx="0.0085" ixy="0.0" ixz="0.0"
+                     iyy="0.0085" iyz="0.0"
+                     izz="0.0006" />
+        </inertial>
+        <visual>
+            <origin xyz="0 0 0" rpy="0 0 0"/>
+            <geometry>
+                <cylinder radius="0.015" length="0.25"/>
+            </geometry>
+            <material name="leg_material">
+                <color rgba="0.4 0.3 0.1 1.0"/>
+            </material>
+        </visual>
+        <collision>
+            <origin xyz="0 0 0" rpy="0 0 0"/>
+            <geometry>
+                <cylinder radius="0.015" length="0.25"/>
+            </geometry>
+        </collision>
+    </link>
+    <link name="metal_object_1">
+        <xacro:default_inertial mass="0.3"/>
+        <visual>
+            <origin xyz="0 0 0" rpy="0 0 0"/>
+            <geometry>
+                <cylinder radius="0.03" length="0.06"/>
+            </geometry>
+            <material name="metal_material_1">
+                <color rgba="0.7 0.7 0.8 1.0"/>
+            </material>
+        </visual>
+        <collision>
+            <origin xyz="0 0 0" rpy="0 0 0"/>
+            <geometry>
+                <cylinder radius="0.03" length="0.06"/>
+            </geometry>
+        </collision>
+    </link>
+    <link name="metal_object_2">
+        <xacro:default_inertial mass="0.25"/>
+        <visual>
+            <origin xyz="0 0 0" rpy="0 0 0"/>
+            <geometry>
+                <box size="0.05 0.05 0.04"/>
+            </geometry>
+            <material name="metal_material_2">
+                <color rgba="0.8 0.8 0.7 1.0"/>
+            </material>
+        </visual>
+        <collision>
+            <origin xyz="0 0 0" rpy="0 0 0"/>
+            <geometry>
+                <box size="0.05 0.05 0.04"/>
+            </geometry>
+        </collision>
+    </link>
     <link name="camera_support_pole">
         <xacro:default_inertial mass="2.0"/>
@@ -201,5 +350,5 @@
             <origin xyz="0 0 0" rpy="0 0 0"/>
             <geometry>
-                <cylinder radius="0.01" length="1.0"/>
+                <cylinder radius="0.01" length="1.2"/>
             </geometry>
             <material name="pole_material">
@@ -210,5 +359,5 @@
             <origin xyz="0 0 0" rpy="0 0 0"/>
             <geometry>
-                <cylinder radius="0.01" length="1.0"/>
+                <cylinder radius="0.01" length="1.2"/>
             </geometry>
         </collision>
@@ -250,9 +399,7 @@
         </collision>
     </link>
-    <!-- Camera optical frame (for ROS conventions) -->
     <link name="camera_optical_frame">
         <xacro:default_inertial mass="0.001"/>
     </link>
-    <!-- Joints -->
     <joint name="virtual_joint" type="fixed">
         <parent link="world"/>
@@ -308,5 +455,4 @@
                effort="${effort}" velocity="${velocity}"/>
     </joint>
-    <!-- Electromagnet Mounting Joints -->
     <joint name="link6_to_electromagnet_mount" type="fixed">
         <parent link="link_6"/>
@@ -319,31 +465,57 @@
         <origin xyz="0 0 0.0175" rpy="0 0 0"/>
     </joint>
-    <!-- Overhead Camera System Joints -->
-    <!-- Support pole mounted to world (positioned above workspace) -->
+ <joint name="world_to_table" type="fixed">
+        <parent link="world"/>
+        <child link="table_base"/>
+        <origin xyz="0.5 0 0.095" rpy="0 0 0"/>
+    </joint>
+    <joint name="table_to_leg_1" type="fixed">
+        <parent link="table_base"/>
+        <child link="table_leg_1"/>
+        <origin xyz="0.22 0.17 -0.095" rpy="0 0 0"/>
+    </joint>
+    <joint name="table_to_leg_2" type="fixed">
+        <parent link="table_base"/>
+        <child link="table_leg_2"/>
+        <origin xyz="-0.22 0.17 -0.095" rpy="0 0 0"/>
+    </joint>
+    <joint name="table_to_leg_3" type="fixed">
+        <parent link="table_base"/>
+        <child link="table_leg_3"/>
+        <origin xyz="0.22 -0.17 -0.095" rpy="0 0 0"/>
+    </joint>
+    <joint name="table_to_leg_4" type="fixed">
+        <parent link="table_base"/>
+        <child link="table_leg_4"/>
+        <origin xyz="-0.22 -0.17 -0.095" rpy="0 0 0"/>
+    </joint>
+   <joint name="table_to_object_1" type="fixed">
+        <parent link="table_base"/>
+        <child link="metal_object_1"/>
+        <origin xyz="-0.18 0.10 0.05" rpy="0 0 0"/>
+    </joint>
+    <joint name="table_to_object_2" type="fixed">
+        <parent link="table_base"/>
+        <child link="metal_object_2"/>
+        <origin xyz="-0.15 -0.08 0.04" rpy="0 0 0"/>
+    </joint>
     <joint name="world_to_camera_pole" type="fixed">
         <parent link="world"/>
         <child link="camera_support_pole"/>
-        <!-- Position pole 0.5m to the side and 1m high -->
-        <origin xyz="0.5 0 1.0" rpy="0 0 0"/>
-    </joint>
-    <!-- Camera mount at top of pole -->
+        <origin xyz="-0.8 0 0.6" rpy="0 0 0"/>
+    </joint>
     <joint name="pole_to_camera_mount" type="fixed">
         <parent link="camera_support_pole"/>
         <child link="camera_mount"/>
-        <!-- Position at top of pole -->
-        <origin xyz="0 0 0.5" rpy="0 0 0"/>
-    </joint>
-    <!-- Camera attached to mount, pointing down at workspace -->
+        <origin xyz="0 0 0.6" rpy="0 0 0"/>
+    </joint>
     <joint name="mount_to_camera" type="fixed">
         <parent link="camera_mount"/>
         <child link="camera_link"/>
-        <!-- Offset slightly and point down -->
-        <origin xyz="0 0 -0.03" rpy="0 ${PI/2} 0"/>
-    </joint>
-    <!-- Camera optical frame for ROS conventions -->
+        <origin xyz="0 0 -0.03" rpy="0 0.5 0"/>
+    </joint>
     <joint name="camera_to_optical_frame" type="fixed">
         <parent link="camera_link"/>
         <child link="camera_optical_frame"/>
-        <!-- Standard ROS camera optical frame transformation -->
         <origin xyz="0 0 0" rpy="-${PI/2} 0 -${PI/2}"/>
     </joint>

File: install/thor_urdf/share/thor_urdf/urdf/thor_gazebo.xacro (robot description, xacro)
@@ -92,4 +92,66 @@
         <material>Gazebo/Orange</material>
     </gazebo>
+   <gazebo reference="table_base">
+        <material>Gazebo/Wood</material>
+        <mu1>0.9</mu1>
+        <mu2>0.9</mu2>
+        <kp>10000000.0</kp>
+        <kd>10.0</kd>
+        <minDepth>0.001</minDepth>
+        <maxVel>0.1</maxVel>
+        <fdir1>0 0 0</fdir1>
+    </gazebo>
+    <gazebo reference="table_leg_1">
+        <material>Gazebo/WoodPallet</material>
+        <mu1>1.0</mu1>
+        <mu2>1.0</mu2>
+        <kp>10000000.0</kp>
+        <kd>100.0</kd>
+        <minDepth>0.001</minDepth>
+        <maxVel>0.01</maxVel>
+    </gazebo>
+    <gazebo reference="table_leg_2">
+        <material>Gazebo/WoodPallet</material>
+        <mu1>1.0</mu1>
+        <mu2>1.0</mu2>
+        <kp>10000000.0</kp>
+        <kd>100.0</kd>
+        <minDepth>0.001</minDepth>
+        <maxVel>0.01</maxVel>
+    </gazebo>
+    <gazebo reference="table_leg_3">
+        <material>Gazebo/WoodPallet</material>
+        <mu1>1.0</mu1>
+        <mu2>1.0</mu2>
+        <kp>10000000.0</kp>
+        <kd>100.0</kd>
+        <minDepth>0.001</minDepth>
+        <maxVel>0.01</maxVel>
+    </gazebo>
+    <gazebo reference="table_leg_4">
+        <material>Gazebo/WoodPallet</material>
+        <mu1>1.0</mu1>
+        <mu2>1.0</mu2>
+        <kp>10000000.0</kp>
+        <kd>100.0</kd>
+        <minDepth>0.001</minDepth>
+        <maxVel>0.01</maxVel>
+    </gazebo>
+    <gazebo reference="metal_object_1">
+        <material>Gazebo/Chrome</material>
+        <mu1>0.3</mu1>
+        <mu2>0.3</mu2>
+        <kp>1000000.0</kp>
+        <kd>1.0</kd>
+        <magnetic_permeability>1000</magnetic_permeability>
+    </gazebo>
+    <gazebo reference="metal_object_2">
+        <material>Gazebo/FlatBlack</material>
+        <mu1>0.4</mu1>
+        <mu2>0.4</mu2>
+        <kp>1000000.0</kp>
+        <kd>1.0</kd>
+        <magnetic_permeability>800</magnetic_permeability>
+    </gazebo>
     <gazebo>
         <plugin name="electromagnet_controller" filename="libgazebo_ros_electromagnet.so">
@@ -103,5 +165,39 @@
             <max_distance>0.05</max_distance>
             <update_rate>100</update_rate>
+            <ferromagnetic_objects>
+                <object>metal_object_1</object>
+                <object>metal_object_2</object>
+            </ferromagnetic_objects>
         </plugin>
+    </gazebo>
+    <gazebo reference="metal_object_1">
+        <sensor name="contact_sensor_obj1" type="contact">
+            <contact>
+                <collision>metal_object_1_collision</collision>
+            </contact>
+            <plugin name="gazebo_ros_contact_sensor" filename="libgazebo_ros_contact_sensor.so">
+                <ros>
+                    <namespace>/thor_arm</namespace>
+                    <remapping>contacts:=metal_object_1/contacts</remapping>
+                </ros>
+                <contact_topic>metal_object_1/contacts</contact_topic>
+                <frame_name>metal_object_1</frame_name>
+            </plugin>
+        </sensor>
+    </gazebo>
+    <gazebo reference="metal_object_2">
+        <sensor name="contact_sensor_obj2" type="contact">
+            <contact>
+                <collision>metal_object_2_collision</collision>
+            </contact>
+            <plugin name="gazebo_ros_contact_sensor" filename="libgazebo_ros_contact_sensor.so">
+                <ros>
+                    <namespace>/thor_arm</namespace>
+                    <remapping>contacts:=metal_object_2/contacts</remapping>
+                </ros>
+                <contact_topic>metal_object_2/contacts</contact_topic>
+                <frame_name>metal_object_2</frame_name>
+            </plugin>
+        </sensor>
     </gazebo>
     <gazebo>
